Commit message: add new launch file

File: urdf/rs200_simulation.xacro (robot description, xacro)
@@ -10,5 +10,5 @@
     <!-- Create camera instance -->
     <xacro:realsense-rs200 prefix="" parent="world">
-        <origin xyz="0 0 1.0" rpy="0 0 0" />
+        <origin xyz="0 0 1.14" rpy="0 0 0" />
     </xacro:realsense-rs200>
 </robot>
